Commit message: Add files via upload

File: bme_gazebo_basics/urdf/mogi_bot.urdf (robot description, URDF)
Before this commit: robot mogi_bot, 4 links, 3 joints
Links:
- link base_link: geometry collision box size=.4 .2 .1; collision sphere radius=0.0499
- link left_wheel: geometry collision cylinder length=.05 radius=.1; visual cylinder length=.05 radius=.1
- link right_wheel: geometry collision cylinder length=.05 radius=.1; visual cylinder length=.05 radius=.1
